Commit message: URDF: actualizar base mas ancha + arreglar nombres snake_case + integrar laser en URDF

File: scr/simulacion_ri/urdf/Ensamblaje_URDF_Final.urdf (robot description, URDF)
Before this commit: robot Ensamblaje_URDF_Final, 7 links, 6 joints
Links:
- removed link base_footprint
- removed link lidar_link
- added link laser, mass 0.141654473640087; collision mesh filename=package://simulacion_ri/meshes/lidar_link.STL; visual mesh filename=package://simulacion_ri/meshes/lidar_link.STL
- link base_link: mass 1.61129016278306 -> 1.62077206884196
- link rueda_delante_derecha_link: mass 0.16695 -> 0.166945647961675
- link rueda_delante_izquierda_link: mass 0.16695 -> 0.166945648004187
- link rueda_trasera_derecha_link: mass 0.16695 -> 0.16694564800895
- link rueda_trasera_izquierda_link: mass 0.16695 -> 0.166945648020152
Joints:
- removed joint base_footprint_joint
- removed joint lidar_joint
- added joint laser_joint: type fixed, parent base_link, child laser, origin xyz=-0.05388 -3.5032E-05 0.17 rpy=0 0 0, axis 0 0 0
- joint rueda_delante_derecha_joint: limit effort=10 velocity=18.85 -> (none); origin xyz=0.090125 -0.14075 0.0125 rpy=0 0 0 -> xyz=0.090145 -0.14075 0.0125 rpy=0 0 0
- joint rueda_delante_izquierda_joint: limit effort=10 velocity=18.85 -> (none); origin xyz=0.090125 0.14065 0.0125 rpy=0 0 0 -> xyz=0.090145 0.14065 0.0125 rpy=0 0 0
- joint rueda_trasera_derecha_joint: limit effort=10 velocity=18.85 -> (none); origin xyz=-0.10111 -0.14075 0.0125 rpy=0 0 0 -> xyz=-0.10109 -0.14075 0.0125 rpy=0 0 0
- joint rueda_trasera_izquierda_joint: limit effort=10 velocity=18.85 -> (none); origin xyz=-0.10111 0.14075 0.0125 rpy=0 0 0 -> xyz=-0.10109 0.14075 0.0125 rpy=0 0 0
